File: no64/no64.kicad_sch (KiCad schematic)
At the start: 16 parts, among them J1 Analog Stick, SW1 A, SW10 Cup, SW11 Cright, SW12 Cdown, SW13 L, SW14 R, SW2 B, SW3 Start, SW4 Dleft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

Commit message: WIP add buttons
Parts:
- removed SW1: A, symbol Switch:SW_MEC_5G
- SW2: value B -> A
- SW3: value Start -> B
- SW8: value L -> START
Connections:
- net GND: now also J1.3 (Pin_3), U1.38 (GND)
- net Cright: now reaches SW11.1 (A), SW11.2 (A)
- net Dup: now reaches SW5.1 (A), SW5.2 (A)
- net R: now reaches SW14.1 (A), SW14.2 (A)
- net Cdown: now reaches SW12.1 (A), SW12.2 (A)
- net L: now reaches SW13.1 (A), SW13.2 (A)
- net Cup: now reaches SW10.1 (A), SW10.2 (A)
- net at U1.3 (GND): no longer J1.3 (Pin_3)
- net 3V3: now reaches J1.2 (Pin_2), U1.36 (3V3)
- net JOY_XA: now reaches J1.1 (Pin_1), U1.4 (GPIO2)
- net JOY_XB: now reaches J1.4 (Pin_4), U1.5 (GPIO3)
- net JOY_YA: now reaches U1.6 (GPIO4)
- net JOY_YA: now also J1.6 (Pin_6); no longer J1.5 (Pin_5)
- net JOY_YB: now reaches U1.7 (GPIO5)
- net JOY_YB: now also J1.5 (Pin_5); no longer J1.6 (Pin_6)
- net B: now reaches SW3.1 (A), SW3.2 (A)
- net Cleft: now reaches SW9.1 (A), SW9.2 (A)
- net Ddown: now reaches SW7.1 (A), SW7.2 (A)
- net Dleft: now reaches SW4.1 (A), SW4.2 (A)
- net Dright: now reaches SW6.1 (A), SW6.2 (A)
- net START: now reaches SW8.1 (A), SW8.2 (A)
- net A: now reaches SW2.1 (A), SW2.2 (A)
Other:
- moved on the sheet: J1, SW13, SW14, SW2, SW3, SW4, SW5, SW6, SW7, SW8
